File: My Projects.kicad_sch (KiCad schematic)
At the start: 87 parts, among them IC1 7483, IC2 7483, IC3 7486, IC4 7486, J1 Barrel_Jack, SW1 SW_SPDT, SW10 SW_SPDT, SW11 SW_SPDT, SW12 SW_SPDT, SW13 SW_SPDT, SW14 SW_SPDT, SW15 SW_SPDT, SW16 SW_SPDT, SW17 SW_Push, SW2 SW_SPDT, SW3 SW_SPDT, SW4 SW_SPDT, SW5 SW_SPDT, SW6 SW_SPDT, SW7 SW_SPDT, SW8 SW_SPDT, SW9 SW_SPDT

Commit message: footprint added
Parts:
- D1, D10, D11, D12, D13, D14, D15, D16, D17, D18, D19, D2, D20, D21, D22, D23, D24, D3, D4, D5, D6, D7, D8, D9: footprint (none) -> LED_THT:LED_D3.0mm
- IC1: footprint Package_DIP:DIP-16_W10.16mm -> Package_DIP:SMDIP-16_W7.62mm
- IC2: footprint (none) -> Package_DIP:SMDIP-16_W7.62mm
- IC3: footprint (none) -> Package_DIP:DIP-14_W7.62mm
- IC4: footprint Package_DIP:DIP-14_W10.16mm -> Package_DIP:DIP-14_W7.62mm
- J1: footprint (none) -> Connector_BarrelJack:BarrelJack_Horizontal
- R1, R10, R11, R12, R13, R14, R15, R16, R17, R18, R19, R2, R20, R21, R22, R23, R24, R25, R26, R27, R28, R29, R3, R30, R31, R32, R33, R34, R35, R36, R37, R38, R39, R4, R40, R41, R5, R6, R7, R8, R9: footprint (none) -> Resistor_THT:R_Axial_DIN0204_L3.6mm_D1.6mm_P5.08mm_Horizontal
- SW17: footprint (none) -> Button_Switch_THT:SW_PUSH_6mm
